File: Hardware/SparkFun GPS RTK Surveyor - Enclosure.sch (EAGLE design)
At the start: 18 parts

Commit message: v13 hardware. Fix power LED. Add gcode for enclosure.
Parts:
- removed D5: Yellow, SparkFun-LED:LED-YELLOW0603
- removed LED2: RED, SparkFun-LED:LED-RED0603
- removed R1, R8: 330, SparkFun-Resistors:330OHM-0603-1/10W-1%
- added B1: 6.8MM_COIN_CELL, SparkFun-Batteries:ML414H_IV01E_BATTERY
- added BLUETOOTH_BROADCAST, SERIAL1_CONNECTION: (no value), SparkFun-Switches:SWITCH-DPDT-SMD-AYZ0202
- added BT1: LIPO-OUTLINE1100, SparkFun-Batteries:LIPO-OUTLINE1100
- added C1: 47pF, SparkFun-Capacitors:47PF-0402-25V-5%-X7R
- added C10, C14: 10uF, SparkFun-Capacitors:10UF-0603-6.3V-20%
- added C11, C12, C13, C15, C16: 0.1uF, SparkFun-Capacitors:0.1UF-0603-25V-(+80/-20%)
- added C2, C3, C4, C6: 1.0uF, SparkFun-Capacitors:1.0UF-0603-16V-10%-X7R
- added C5, C7: 0.1uF, SparkFun-Capacitors:0.1UF-0603-25V-5%
- added C8, C9: 4.7uF, SparkFun-Capacitors:4.7UF-0603-35V-(20%)
- added D13: RGB, SparkFun-LED:LED-RGB-CAPLCC
- added D2: 0.5A/40V/420mV, SparkFun-DiscreteSemi:DIODE-SCHOTTKY-PMEG4005EJ
- added D6: PRTR5V0U2F, SparkFun-IC-Power:PRTR5V0U2F
- added D7, D9: 3A/10V/280mV, SparkFun-DiscreteSemi:DIODE-SCHOTTKY-BAT60A
- added DUAL_OUTPUT: JUMPER-SMT_2_NO_SILK, SparkFun-Jumpers:JUMPER-SMT_2_NO_SILK
- added E1: SMA, SparkFun-RF:ANTENNA-GROUNDEDEDGE_SMA_SMD
- added FB1: 2.66Ω, SparkFun-Coils:FERRITE_BEAD-0402-2.66OHM-1GHZ
- added J1, J11, J12, J13: (no value), SparkFun-Connectors:CONN_041X04_NO_SILK_NO_POP
- added J10, J14, J15: (no value), SparkFun-Connectors:CONN_021X02_NO_SILK
- added J16: microSD, SparkFun-Connectors:MICRO-SD-SDIOPUSH-PUSH
- added J2, J9: (no value), SparkFun-Connectors:CONN_04JST-SMD-LOCKING
- added J3: USB-C, SparkFun-Connectors:USB_C_2-LAYER_PADS
- added J4: Qwiic Right Angle, SparkFun-Connectors:I2C_STANDARDQWIIC
- added J5: (no value), SparkFun-Connectors:USB_C_2-LAYER_PADS
- added J6: Start Base, SparkFun-Connectors:CONN_02-JST-2MM-SMT
- added J7: Power Switch, SparkFun-Connectors:CONN_02-JST-2MM-SMT
- added J8: (no value), SparkFun-Connectors:JST_2MM_MALE
- added JP21, JP61, JP71, JP81: FIDUCIALUFIDUCIAL, SparkFun-Aesthetics:FIDUCIALUFIDUCIAL
- added LOGO1: OSHW-LOGOMINI, SparkFun-Aesthetics:OSHW-LOGOMINI
- added LOGO2: SFE_LOGO_NAME_FLAME.1_INCH, SparkFun-Aesthetics:SFE_LOGO_NAME_FLAME.1_INCH
- added MEAS, MEAS1: JUMPER-COMBO_2_NC_TRACE, SparkFun-Jumpers:JUMPER-COMBO_2_NC_TRACE
- added Q2: MBT3904DW1T1, SparkFun-DiscreteSemi:TRANS_NPN_DUAL-MBT3904DW1T1
- added R13, R15: 100k, SparkFun-Resistors:100KOHM-0603-1/10W-1%
- added R14: 10, SparkFun-Resistors:10OHM-0603-1/10W-1%
- added R16, R17, R37, R38: 5.1k, SparkFun-Resistors:5.1KOHM5.1KOHM-0603-1/10W-1%
- added R2, R4, R9: 33, SparkFun-Resistors:33OHM_RA-1206-1/16W-5%
- added R20, R23, R29: 10k, SparkFun-Resistors:10KOHM-0603-1/10W-1%
- added R27, R28: 27, SparkFun-Resistors:27OHM-0603-1/10W-1%
- added R3: 33, SparkFun-Resistors:33OHM-0603-1/10W-1%
- added R5: 3.3k, SparkFun-Resistors:3.3KOHM-0603-1/10W-1%
- added R7: 1k, SparkFun-Resistors:1KOHM-0603-1/10W-1%
- added S1: RESET, SparkFun-Switches:MOMENTARY-SWITCH-SPST-SMD-5.2-TALL-REDUNDANT
- added U1: MCP73831, SparkFun-IC-Power:MCP73831
- added U2: 3.3V, SparkFun-IC-Power:V_REG_AP2112K-3.3V
- added U3: U-BLOX_ZED-F9P, SparkFun-GPS:U-BLOX_ZED-F9P
- added U5: ESP-WROOM-32NARROW, SparkFun-RF:ESP-WROOM-32NARROW
- added U6: CH340C, SparkFun-IC-Comms:CH340C
- added U7: MAX17048, SparkFun-IC-Power:MAX17048DFN8
Connections:
- removed net ESP32_12/BLUETOOTH_STATUS: R10.1
- removed net ESP32_13/POSACC3: R24.1
- removed net ESP32_15/POSACC2: R25.1
- removed net ESP32_2/POSACC1: R26.1
- removed net ESP32_4/BASE_STAT: R34.1
- removed net N$10: LED2.A, R1.1
- removed net N$8: D5.C, R8.2
- removed net PPS_STAT: R11.2
- removed net RTK_STAT: D3.C
- new net 5V: C6.1, J11.4, J7.2, J9.1, U2.EN, U2.IN
- new net ANT_VCC: C1.1, FB1.2, R14.1
- new net BACKUP: B1.+, C3.1, R5.1, U3.V_BKCP
- new net CC1: J5.CC1, R17.2
- new net CC2: J5.CC2, R16.2
- new net CC3: J3.CC2, R37.2
- new net CC4: J3.CC1, R38.2
- new net D+: D6.4, R27.1
- new net D+1: J3.D+, U6.UD+
- new net D-: D6.6, R28.1
- new net D-1: J3.D-, U6.UD-
- new net ESP32_!DTR: Q2Q2.E, R23.1, U6.!DTR
- new net ESP32_!RTS: Q2Q1.E, R29.1, U6.!RTS
- new net ESP32_EN: C12.1, Q2Q1.C, R20.1, S1.2, U5.EN
- new net ESP32_RXI: U5.RXD, U6.TXO
- new net ESP32_TXO: U5.TXD, U6.RXI
- new net ESP_0/BOOT: Q2Q2.C, U5.IO0
- new net ESP_12/LED_BLUETOOTH: R10.1, U5.MISO_H/IO12
- new net ESP_13/LED_100CM: R24.1, U5.MOSI_H/IO13
- new net ESP_14: U5.SCK_H/IO14
- new net ESP_15/LED_10CM: R25.1, U5.CS0_H/IO15
- new net ESP_16/BT_RXI: BLUETOOTH_BROADCAST.5, U5.IO16
- new net ESP_17/BT_TXO: BLUETOOTH_BROADCAST.2, U5.IO17
- new net ESP_18/SD_SCK: J16.CLK/SCK, U5.SCK_V/IO18
- new net ESP_19/SD_CIPO: J16.DAT0/SDO, U5.MISO_V/IO19
- new net ESP_2/LED_1CM: R26.1, U5.IO2
- new net ESP_21/SDA: J4.3, R9C.2, U5.IO21, U7.SDA
- new net ESP_22/SCL: J4.4, R9B.2, U5.IO22, U7.SCL
- new net ESP_23/SD_COPI: J16.CMD/SDI, U5.MOSI_V/IO23
- new net ESP_25/SD_!CS!: J16.DAT3/!CS!, R13.1, U5.IO25
- new net ESP_26/ZED_TX_READY: J13.4, R9A.2, U5.IO26
- new net ESP_27/ZED_!RESET!: J13.3, R2D.2, U5.IO27
- new net ESP_32: J14.2, U5.XTAL_P/IO32
- new net ESP_33: J14.1, U5.XTAL_N/IO33
- new net ESP_34/PWR_LVL_RED: D13.RED, U5.IO34
- new net ESP_35/PWR_LVL_GRN: D13.GRN, U5.IO35
- new net ESP_36/BATT_ALRT: U5.SENSOR_VP/I36, U7.!ALRT
- new net ESP_4/LED_BASE_STAT: R34.1, U5.IO4
- new net ESP_5/SWITCH_BASE_SELECT: J6.2, U5.CS0_V/IO5
- new net ESP_I39: U5.SENSOR_VN/I39
- new net EXTERNAL_SERIAL1_RXI: J12.2, J2.3, SERIAL1_CONNECTION.3
- new net EXTERNAL_SERIAL1_TXO: DUAL_OUTPUT.2, J12.3, J2.2, SERIAL1_CONNECTION.6
- new net FENCE_LV: R4A.2, U3.GEO_STAT
- new net GPS_ANT1: E1.SIGNAL, FB1.1, U3.RF_IN
- new net N$11: R27.2, U3.USB_D+
- new net N$12: R28.2, U3.USB_D-
- new net N$13: R14.2, U3.V_RF
- new net N$16: R2D.1, U3.!RESET!
- new net N$18: R2C.1, U3.!SAFEBOOT!
- new net N$22: R9A.1, U3.TX_READY
- new net N$24: Q2Q1.B, R23.2
- new net N$25: Q2Q2.B, R29.2
- new net N$32: D9.A, J3.VBUS
- new net N$4: J5.VBUS, MEAS.1
- new net N$5: R7.2, U1.PROG
- new net N$6: D2.C, R5.2
- new net N$7: J8.+, MEAS1.1
- new net NMEA-RX: BLUETOOTH_BROADCAST.1, SERIAL1_CONNECTION.1
- new net NMEA-TX: BLUETOOTH_BROADCAST.4, DUAL_OUTPUT.1, SERIAL1_CONNECTION.4
- new net PPS: R2A.1, U3.TIMEPULSE
- new net RTK_LV: R4B.2, U3.RTK_STAT
- new net RX2_LV: R4C.2, U3.RX2
- new net RXLV: R9D.1, U3.RX/MOSI
- new net SCL_LV: R9B.1, U3.SCL/CLK
- new net SDA_LV: R9C.1, U3.SDA/!CS!
- new net TX2_LV: R4D.2, U3.TX2
- new net TXLV: R3.1, U3.TX/MISO
- new net UNP_D+: D6.3, J5.D+
- new net UNP_D-: D6.1, J5.D-
- new net V_BATT: C15.1, C8.1, D7.A, J10.1, MEAS1.2, U1.VBAT, U7.CELL, U7.VDD
- new net ZED-RXI1: J15.2, R9D.2, SERIAL1_CONNECTION.2
- new net ZED-RXI2: BLUETOOTH_BROADCAST.3, J11.2, J9.3, R4C.1
- new net ZED-TXO1: J15.1, R3.2, SERIAL1_CONNECTION.5
- new net ZED-TXO2: BLUETOOTH_BROADCAST.6, J11.3, J9.2, R4D.1
- new net ZED_!SAFE!: J13.2, R2C.2
- new net ZED_FENCE_STAT: J1.2, R4A.1
- new net ZED_PPS_STAT: J13.1, R11.2, R2A.2
- new net ZED_RTK_STAT: D3.C, J1.3, R4B.1
- net 3.3V: now also C10.1, C11.1, C13.1, C14.1, C16.1, C2.1, C4.1, C5.2, C7.2, D2.A, J1.4, J12.4, J16.VCC, J2.1, J4.2, R13.2, R15.2, R20.2, U2.OUT, U3.VCC, U3.V_USB, U5.3V3, U6.V3, U6.VCC; no longer R1.2
- net CHG_LED: now also D13.BLU, U1.STAT; no longer R8.1
- net GND: now also B1.-, C1.2, C10.2, C11.2, C12.2, C13.2, C14.2, C15.2, C16.2, C2.2, C3.2, C4.2, C5.1, C6.2, C7.1, C8.2, C9.2, D6.2, E1.GND, J1.1, J10.2, J11.1, J12.1, J16.GND, J16.SHIELD, J2.4, J3.GND, J3.SHLD, J4.1, J5.GND, J5.SHLD, J6.1, J8.-, J9.4, R15.1, R16.1, R17.1, R37.1, R38.1, R7.1, S1.1, U1.VSS, U2.GND, U3.GND, U5.GND, U6.GND, U7.CTG, U7.GND, U7.QSTRT; no longer LED2.C
- net VIN: now also C9.1, D13.A, D6.5, D7.C, D9.C, J7.1, MEAS.2, U1.VIN; no longer D5.A
Other:
- note added: "5V is not guaranteed May be 3.5-5V"
- note added: "7-bit unshifted I2C address: 0x42"
- note added: "Bluetooth"
- note added: "Board thickness: 1.6mm"
- note added: "Charge current: 1000mA (1000V/Rprog)"
- note added: "Close DUAL_OUTPUT jumper to output NMEA Serial1 to both Bluetooth and external Serial1 port."
- note added: "Connections"
- note added: "Copper Thickness (1oz): 1.4mil/0.035mm"
- note added: "Data Output Selection"
- note added: "Default: Bluetooth will broadcast NMEA. Move switch to 'RTCM' to use Bluetooth as radio connection between RTK units for RTCM corrections."
- note added: "Default: ZED-Serial1 NMEA connected to Bluetooth. Move switch to 'Ext Cntr' to connect external 'Data' connector to ZED-Serial1."
- note added: "Dielectric thickness (layer 1 to 2): 0.2mm"
- note added: "ESP32-WROOM"
- note added: "Er: 4.6"
- note added: "External Radio RTCM In/Out"
- note added: "Fuel Gauge"
- note added: "LQW15ANR12J00D"
- note added: "LiPo Charger"
- note added: "LiPo Range: 3.6-4.2V"
- note added: "Microstrip Calculation:"
- note added: "NMEA"
- note added: "No clean process"
- note added: "Polygon Isolation: 8mil/0.2032mm"
- note added: "RF Trace Width: 13.8mil/0.35mm"
- note added: "RTC Backup"
- note added: "RTCM"
- note added: "Serial Config NMEA Out"
- note added: "USB / Power"
- note added: "USB-to-Serial For ESP32"
- note added: "Ublox ZED-F9P"
- note added: "https://chemandy.com/calculators/coplanar-waveguide-with-ground-calculator.htm"
- note added: "v12"
- note added: "μSD"
- moved on the sheet: D1, D3, R11, R12
