File: Hardware/SparkFun GPS RTK Surveyor.sch (EAGLE design)
At the start: 122 parts, among them J13 Internal, J16 microSD, J17 Qwiic Right Angle, J3 USB Female Type C Connector, J4 External, J5 USB Female Type C Connector, Q1 SIL2308-TP, Q10 20V/0.2A/8MHz/1.2Ω/1Vth, Q2 MBT3904DW1T1, Q3 20V/0.2A/8MHz/1.2Ω/1Vth, Q4 20V/0.2A/8MHz/1.2Ω/1Vth, Q7 20V/0.2A/8MHz/1.2Ω/1Vth, Q9 20V/0.2A/8MHz/1.2Ω/1Vth, U1 74HC4052D, U10 MCP73833, U13 9DoF IMU, U14 1.8V/100mA, U2 AP2112K-3.3, U3 U-BLOX_ZED-F9P, U4 ADP160, U5 ESP-WROOM-32NARROW, U6 CH340C, U7 MAX17048

Commit message: Revert hardware files back to v15
Parts:
- removed C20: 10uF, SparkFun-Capacitors:10UF-0603-6.3V-20%
- removed C22, C23: 0.1uF, SparkFun-Capacitors:0.1UF-0603-25V-5%
- removed C3, C52: 0.1uF, SparkFun-Capacitors:0.1UF-0603-25V-(+80/-20%)
- removed C51: 0.1uF, SparkFun-Capacitors:0.1UF-0603-100V-10%
- removed C53, C54: 1.0uF, SparkFun-Capacitors:1.0UF-0603-16V-10%
- removed Q1: SIL2308-TP, SparkFun-DiscreteSemi:MOSFET_COMPLIMENTARY_PAIR-SIL2308
- removed Q10, Q3, Q4, Q7, Q9: 20V/0.2A/8MHz/1.2Ω/1Vth, SparkFun-DiscreteSemi:MOSFET-NCH-RE1C00UNTL
- removed R19: 1k, SparkFun-Resistors:1KOHM-0603-1/10W-1%
- removed R22: 100k, SparkFun-Resistors:100KOHM-0603-1/10W-1%
- removed R31: 10k, SparkFun-Resistors:10KOHM-0603-1/10W-1%
- removed R40, R41, R44, R45, R46, R47, R48: 2.2k, SparkFun-Resistors:2.2KOHM-0603-1/10W-1%
- removed R49: (no value), SparkFun-Resistors:RESISTOR0603
- removed S1: Power, SparkFun-Switches:MOMENTARY-SWITCH-SPST-PTH-6.0MM
- removed S2: Setup, SparkFun-Switches:MOMENTARY-SWITCH-SPST-PTH-6.0MM
- removed S3: Power, SparkFun-Switches:MOMENTARY-SWITCH-SPST-SMD-12MM
- removed S4: Setup, SparkFun-Switches:MOMENTARY-SWITCH-SPST-SMD-12MM
- removed U1: 74HC4052D, SparkFun-IC-Logic:74HC4052D
- removed U13: 9DoF IMU, SparkFun-Sensors:ICM-20948
- removed U14: 1.8V/100mA, SparkFun-IC-Power:V_REG_SP6214-1.8V
- added BLUETOOTH_BROADCAST, SERIAL1_CONNECTION, ZED_CONTROL: (no value), SparkFun-Switches:SWITCH-DPDT-SMD-AYZ0202
- added D10, D11, D8: GREEN, SparkFun-LED:LED-GREEN0603
- added D12: RED, SparkFun-LED:LED-RED0603
- added DUAL_OUTPUT: JUMPER-SMT_2_NO_SILK, SparkFun-Jumpers:JUMPER-SMT_2_NO_SILK
- added J18: (no value), SparkFun-Connectors:CONN_05NO_SILK
- added R11, R25: 20, SparkFun-Resistors:20OHM-0603-1/10W-1%
- added R12, R34: 330, SparkFun-Resistors:330OHM-0603-1/10W-1%
- D1: value 250mA/100V -> Yellow; device SparkFun-DiscreteSemi:DIODE-BAS16J -> SparkFun-LED:LED-YELLOW0603
- D3: value 3A/10V/280mV -> WHITE; device SparkFun-DiscreteSemi:DIODE-SCHOTTKY-BAT60A -> SparkFun-LED:LED-WHITE0603
- J6: value (none) -> Start Base; device SparkFun-Connectors:CONN_05NO_SILK -> SparkFun-Connectors:CONN_02-JST-2MM-SMT
- J7: value (none) -> Power Switch; device SparkFun-Connectors:CONN_041X04_NO_SILK_NO_POP -> SparkFun-Connectors:CONN_02-JST-2MM-SMT
- R20: value 100k -> 10k; device SparkFun-Resistors:100KOHM-0603-1/10W-1% -> SparkFun-Resistors:10KOHM-0603-1/10W-1%
- R24: value 300k -> 20; device SparkFun-Resistors:300KOHM-0603-1/10W-1% -> SparkFun-Resistors:20OHM-0603-1/10W-1%
- R26: value 100k -> 20; device SparkFun-Resistors:100KOHM-0603-1/10W-1% -> SparkFun-Resistors:20OHM-0603-1/10W-1%
- R3: device SparkFun-Resistors:33OHM_RA-1206-1/16W-5% -> SparkFun-Resistors:33OHM-0603-1/10W-1%
- U2: value AP2112K-3.3 -> 3.3V
- U4: value ADP160 -> 3.3V; device SparkFun-IC-Power:ADP160 -> SparkFun-IC-Power:V_REG_AP2112K-3.3V
Connections:
- net RTC_BACKUP renamed BACKUP
- removed net CHG_LED_RES: D5.BLU-C, J7.2, R1.1
- removed net ESP_13/POWER_CTRL: D1.A, R22.1, R24.2, U5.MOSI_H/IO13
- removed net ESP_14/SETUP_BUTTON: J7.3, S2.1, S4.1, U5.SCK_H/IO14
- removed net ESP_15/ICM_!CS!: Q9.D, R47.1, U5.CS0_H/IO15
- removed net ESP_18/SCK: J16.CLK/SCK, Q3.D, U5.SCK_V/IO18
- removed net ESP_19/CIPO: J16.DAT0/SDO, Q10.D, R49.1, U5.MISO_V/IO19
- removed net ESP_2/MUX_A: U1.A, U5.IO2
- removed net ESP_23/COPI: J16.CMD/SDI, Q4.D, U5.MOSI_V/IO23
- removed net ESP_26/DAC2: U1.X3, U5.IO26
- removed net ESP_27: U5.IO27
- removed net ESP_4/MUX_B: U1.B, U5.IO4
- removed net ESP_5: U5.CS0_V/IO5
- removed net ESP_I16/ZED-TXO1: J15.1, R2D.2, U1.X0, U5.IO16
- removed net ESP_I34/ZED_TX_READY: J6.1, R3D.2, U5.I34
- removed net ESP_I36/ICM_INT: Q7.D, R45.1, U5.SENSOR_VP/I36
- removed net ESP_I39/ADC39: U1.Y3, U5.SENSOR_VN/I39
- removed net ESP_O17/ZED-RXI1: J15.2, R19.2, R2C.2, U1.Y0
- removed net EXTERNAL_DATA_IN: J12.2, J2.3, U1.Y
- removed net EXTERNAL_DATA_OUT: J12.3, J2.2, U1.X
- removed net EXTINT_LV: R9B.1, U3.EXTINT
- removed net ICM-20948-LV_!CS!: Q9.S, R46.1, U13.!CS
- removed net ICM-20948-LV_#_1.8V: C52.1, C53.1, Q10.G, Q3.G, Q4.G, Q7.G, Q9.G, R40.2, R41.2, R44.2, R46.2, R48.2, U13.VDD, U13.VDDIO, U14.OUT
- removed net ICM-20948-LV_INT: Q7.S, R44.1, U13.INT
- removed net ICM-20948-LV_SCK: Q3.S, R40.1, U13.SCL/SCLK
- removed net ICM-20948-LV_SDI: Q4.S, R41.1, U13.SDA/SDI
- removed net ICM-20948-LV_SDO: Q10.S, R48.1, U13.AD0/SDO
- removed net N$15: C22.1, C23.2, Q1G1.D, Q1G2.G, R26.1
- removed net N$6: R19.1, U5.IO17
- removed net N$8: C20.2, Q1G1.G, R24.1
- removed net POWER_BTN: C23.1, D1.C, J7.4, R31.1, S1.1, S3.1
- removed net VOUT: C20.1, C6.1, Q1G2.D, R22.2, U2.EN, U2.IN
- removed net V_RAW: C22.2, C9.1, D3.C, D7.C, J11.4, J9.1, Q1G2.S, R26.2, R31.2, U10.VDD
- removed net V_USB: D2.5, D3.A, D5.BLU-A, D6.5, D9.C, MEAS.2
- removed net ZED_!RESET!: J6.3, R3B.2
- removed net ZED_!RESET!_LV: R3B.1, U3.!RESET!
- removed net ZED_EXTINT: R9B.2, U1.Y1
- new net 5V: C6.1, J11.4, J7.2, J9.1, U2.EN, U2.IN
- new net ESP_13/LED_100CM: R24.1, U5.MOSI_H/IO13
- new net ESP_14: U5.SCK_H/IO14
- new net ESP_15/LED_10CM: R25.1, U5.CS0_H/IO15
- new net ESP_16/BT_RXI: BLUETOOTH_BROADCAST.2, U5.IO16
- new net ESP_17/BT_TXO: BLUETOOTH_BROADCAST.5, U5.IO17
- new net ESP_18/SD_SCK: J16.CLK/SCK, U5.SCK_V/IO18
- new net ESP_19/SD_CIPO: J16.DAT0/SDO, U5.MISO_V/IO19
- new net ESP_2/LED_1CM: R26.1, U5.IO2
- new net ESP_23/SD_COPI: J16.CMD/SDI, U5.MOSI_V/IO23
- new net ESP_26/ZED_TX_READY: J18.1, R9A.2, U5.IO26
- new net ESP_27/ZED_!RESET!: J18.2, R2D.2, U5.IO27, ZED_CONTROL.4
- new net ESP_27/ZED_!RESET!_LV: R2D.1, U3.!RESET!
- new net ESP_36/BATT_ALRT: U5.SENSOR_VP/I36, U7.!ALRT
- new net ESP_4/LED_BASE_STAT: R34.1, U5.IO4
- new net ESP_5/SWITCH_BASE_SELECT: J6.2, U5.CS0_V/IO5
- new net ESP_I34: U5.I34
- new net ESP_I39: U5.SENSOR_VN/I39
- new net EXTERNAL_SERIAL1_RXI: SERIAL1_CONNECTION.4, ZED_CONTROL.6
- new net EXTERNAL_SERIAL1_RXI/ZED_!RESET!: J12.2, J2.3, ZED_CONTROL.5
- new net EXTERNAL_SERIAL1_TXO: DUAL_OUTPUT.2, SERIAL1_CONNECTION.1, ZED_CONTROL.3
- new net EXTERNAL_SERIAL1_TXO/PPS: J12.3, J2.2, ZED_CONTROL.2
- new net N$1: D3.A, R12.1
- new net N$17: D5.BLU-C, R1.1
- new net N$2: D1.A, R11.1
- new net N$26: D8.A, R24.2
- new net N$27: D10.A, R25.2
- new net N$29: D11.A, R26.2
- new net NMEA-RX: BLUETOOTH_BROADCAST.6, SERIAL1_CONNECTION.6
- new net NMEA-TX: BLUETOOTH_BROADCAST.3, DUAL_OUTPUT.1, SERIAL1_CONNECTION.3
- new net VIN: C9.1, D2.5, D5.BLU-A, D6.5, D7.C, D9.C, J7.1, MEAS.2, U10.VDD
- new net ZED-RXI1: J15.2, R9D.2, SERIAL1_CONNECTION.5
- new net ZED-TXO1: J15.1, R3.2, SERIAL1_CONNECTION.2
- net 3.3V: now also R12.2; no longer C3.1, C54.1, R45.2, R47.2, R49.2, U1.VCC, U14.EN, U14.IN
- net ESP_21/SDA: now also R9C.2; no longer R2B.2, U1.Y2
- net ESP_22/SCL: now also R9B.2; no longer R2A.2, U1.X2
- net ESP_26/ZED_TX_READY_LV: now also R9A.1; no longer R3D.1
- net FENCE_LV: now also R4A.2; no longer R4D.1
- net GND: now also D1.C, D10.C, D11.C, D12.C, D8.C, J6.1; no longer C3.2, C51.2, C52.2, C53.2, C54.2, J7.1, Q1G1.S, S1.2, S2.2, S3.2, S4.2, U1.GND, U1.INH, U1.VEE, U13.GND, U14.GND
- net N$30: now also D12.A, R34.2; no longer C51.1, U13.REGOUT
- net PPS: now also R2A.1; no longer R9A.1
- net RTK_LV: now also R4B.2; no longer R4C.1
- net RX2_LV: now also R4C.2; no longer R4B.1
- net RXLV: now also R9D.1; no longer R2C.1
- net SCL_LV: now also R9B.1; no longer R2A.1
- net SDA_LV: now also R9C.1; no longer R2B.1
- net TX2_LV: now also R4D.2; no longer R4A.1
- net TXLV: now also R3.1; no longer R2D.1
- net ZED-RXI2: now also BLUETOOTH_BROADCAST.4, R4C.1; no longer R4B.2
- net ZED-TXO2: now also BLUETOOTH_BROADCAST.1, R4D.1; no longer R4A.2
- net ZED_!SAFE!: now also J18.3, R2C.2; no longer J6.4, R3A.2
- net ZED_!SAFE!_LV: now also R2C.1; no longer R3A.1
- net ZED_D_SEL: now also J18.5, R2B.2; no longer J6.2, R3C.2
- net ZED_D_SEL_LV: now also R2B.1; no longer R3C.1
- net ZED_FENCE_STAT: now also R4A.1; no longer R4D.2
- net ZED_PPS_STAT: now also J18.4, R11.2, R2A.2, ZED_CONTROL.1; no longer J6.5, R9A.2, U1.X1
- net ZED_RTK_STAT: now also D3.C, R4B.1; no longer R4C.2
Other:
- note added: "Base Status"
- note added: "Bluetooth"
- note added: "Close DUAL_OUTPUT jumper to output NMEA Serial1 to both Bluetooth and external Serial1 port."
- note added: "Default: Bluetooth will broadcast NMEA. Move switch to 'RTCM' to use Bluetooth as radio connection between RTK units for RTCM corrections."
- note added: "Default: Data Port Outputs Serial/NMEA Move switch to 'PPS/Reset' to connect Pulse-Per-Second to TX pin and ZED-Reset to RX pin"
- note added: "Default: ZED-Serial1 NMEA connected to Bluetooth. Move switch to 'Ext Cntr' to connect external 'Data' connector to ZED-Serial1."
- note added: "Ext Cntr"
- note added: "NMEA"
- note added: "PPS/Reset"
- note added: "RTCM"
- note added: "RTK Solution: Off: None Blinking: Float On: Fixed"
- note added: "Serial Config NMEA Out"
- note added: "Serial NMEA"
- note added: "USB For ZED-F9P Power Switch"
- note added: "Ublox ZED-F9P"
- note added: "≤1000mm"
- note added: "≤100mm"
- note added: "≤20mm"
- note removed: "3uA Hibernate"
- note removed: "600mA Max 55uA Quiescent"
- note removed: "80uA Quiescent"
- note removed: "860nA Quiescent"
- note removed: "Controller In Peripheral Out (CIPO)"
- note removed: "Controller Out Peripheral In (COPI)"
- note removed: "External Data Port"
- note removed: "ICM-20948 IMU"
- note removed: "Level Shifting"
- note removed: "Maintains GNSS data/almanac"
- note removed: "Power Select"
- note removed: "R19 prevents potential serial contention with Data Port"
- note removed: "SP6214-1.8V ---------------- Iout (max): 100mA Vin (max): 7.0V Vdrop (max): 250mV Iq: 65uA"
- note removed: "System Power"
- note removed: "USB For ZED-F9P"
- note removed: "Voltage Regulator"
- note removed: "u-blox ZED-F9P"
- moved on the sheet: C17, C18, C4, C5, C6, C8, C9, D4, D5, D6, D7, J10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

Commit message: Implement soft power control. Add overlay connection.
Parts:
- removed BLUETOOTH_BROADCAST, SERIAL1_CONNECTION, ZED_CONTROL: (no value), SparkFun-Switches:SWITCH-DPDT-SMD-AYZ0202
- removed D10, D11, D8: GREEN, SparkFun-LED:LED-GREEN0603
- removed D12: RED, SparkFun-LED:LED-RED0603
- removed DUAL_OUTPUT: JUMPER-SMT_2_NO_SILK, SparkFun-Jumpers:JUMPER-SMT_2_NO_SILK
- removed J18: (no value), SparkFun-Connectors:CONN_05NO_SILK
- removed R11, R25: 20, SparkFun-Resistors:20OHM-0603-1/10W-1%
- removed R12, R34: 330, SparkFun-Resistors:330OHM-0603-1/10W-1%
- added C20: 10uF, SparkFun-Capacitors:10UF-0603-6.3V-20%
- added C22, C23: 0.1uF, SparkFun-Capacitors:0.1UF-0603-25V-5%
- added C3, C52: 0.1uF, SparkFun-Capacitors:0.1UF-0603-25V-(+80/-20%)
- added C51: 0.1uF, SparkFun-Capacitors:0.1UF-0603-100V-10%
- added C53, C54: 1.0uF, SparkFun-Capacitors:1.0UF-0603-16V-10%
- added Q1: DMC2700UDM, SparkFun-DiscreteSemi:MOSFET_COMPLIMENTARY_PAIR-DMC2700UDM
- added Q10, Q3, Q4, Q7, Q9: 20V/0.2A/8MHz/1.2Ω/1Vth, SparkFun-DiscreteSemi:MOSFET-NCH-RE1C00UNTL
- added R19: 1k, SparkFun-Resistors:1KOHM-0603-1/10W-1%
- added R22: 100k, SparkFun-Resistors:100KOHM-0603-1/10W-1%
- added R31: 10k, SparkFun-Resistors:10KOHM-0603-1/10W-1%
- added R40, R41, R44, R45, R46, R47, R48: 2.2k, SparkFun-Resistors:2.2KOHM-0603-1/10W-1%
- added R49: (no value), SparkFun-Resistors:RESISTOR0603
- added S1: Power, SparkFun-Switches:MOMENTARY-SWITCH-SPST-PTH-6.0MM
- added S2: Setup, SparkFun-Switches:MOMENTARY-SWITCH-SPST-PTH-6.0MM
- added S3: Power, SparkFun-Switches:MOMENTARY-SWITCH-SPST-SMD-12MM
- added S4: Setup, SparkFun-Switches:MOMENTARY-SWITCH-SPST-SMD-12MM
- added U1: 74HC4052D, SparkFun-IC-Logic:74HC4052D
- added U13: 9DoF IMU, SparkFun-Sensors:ICM-20948
- added U14: 1.8V/100mA, SparkFun-IC-Power:V_REG_SP6214-1.8V
- D1: value Yellow -> 250mA/100V; device SparkFun-LED:LED-YELLOW0603 -> SparkFun-DiscreteSemi:DIODE-BAS16J
- D3: value WHITE -> 3A/10V/280mV; device SparkFun-LED:LED-WHITE0603 -> SparkFun-DiscreteSemi:DIODE-SCHOTTKY-BAT60A
- J6: value Start Base -> (none); device SparkFun-Connectors:CONN_02-JST-2MM-SMT -> SparkFun-Connectors:CONN_05NO_SILK
- J7: value Power Switch -> (none); device SparkFun-Connectors:CONN_02-JST-2MM-SMT -> SparkFun-Connectors:CONN_041X04_NO_SILK_NO_POP
- R20: value 10k -> 100k; device SparkFun-Resistors:10KOHM-0603-1/10W-1% -> SparkFun-Resistors:100KOHM-0603-1/10W-1%
- R24: value 20 -> 300k; device SparkFun-Resistors:20OHM-0603-1/10W-1% -> SparkFun-Resistors:300KOHM-0603-1/10W-1%
- R26: value 20 -> 100k; device SparkFun-Resistors:20OHM-0603-1/10W-1% -> SparkFun-Resistors:100KOHM-0603-1/10W-1%
- R3: device SparkFun-Resistors:33OHM-0603-1/10W-1% -> SparkFun-Resistors:33OHM_RA-1206-1/16W-5%
- U2: value 3.3V -> AP2112K-3.3
- U4: value 3.3V -> ADP160; device SparkFun-IC-Power:V_REG_AP2112K-3.3V -> SparkFun-IC-Power:ADP160
Connections:
- net BACKUP renamed RTC_BACKUP
- removed net 5V: C6.1, J11.4, J7.2, J9.1, U2.EN, U2.IN
- removed net ESP_13/LED_100CM: R24.1, U5.MOSI_H/IO13
- removed net ESP_14: U5.SCK_H/IO14
- removed net ESP_15/LED_10CM: R25.1, U5.CS0_H/IO15
- removed net ESP_16/BT_RXI: BLUETOOTH_BROADCAST.2, U5.IO16
- removed net ESP_17/BT_TXO: BLUETOOTH_BROADCAST.5, U5.IO17
- removed net ESP_18/SD_SCK: J16.CLK/SCK, U5.SCK_V/IO18
- removed net ESP_19/SD_CIPO: J16.DAT0/SDO, U5.MISO_V/IO19
- removed net ESP_2/LED_1CM: R26.1, U5.IO2
- removed net ESP_23/SD_COPI: J16.CMD/SDI, U5.MOSI_V/IO23
- removed net ESP_26/ZED_TX_READY: J18.1, R9A.2, U5.IO26
- removed net ESP_27/ZED_!RESET!: J18.2, R2D.2, U5.IO27, ZED_CONTROL.4
- removed net ESP_27/ZED_!RESET!_LV: R2D.1, U3.!RESET!
- removed net ESP_36/BATT_ALRT: U5.SENSOR_VP/I36, U7.!ALRT
- removed net ESP_4/LED_BASE_STAT: R34.1, U5.IO4
- removed net ESP_5/SWITCH_BASE_SELECT: J6.2, U5.CS0_V/IO5
- removed net ESP_I34: U5.I34
- removed net ESP_I39: U5.SENSOR_VN/I39
- removed net EXTERNAL_SERIAL1_RXI: SERIAL1_CONNECTION.4, ZED_CONTROL.6
- removed net EXTERNAL_SERIAL1_RXI/ZED_!RESET!: J12.2, J2.3, ZED_CONTROL.5
- removed net EXTERNAL_SERIAL1_TXO: DUAL_OUTPUT.2, SERIAL1_CONNECTION.1, ZED_CONTROL.3
- removed net EXTERNAL_SERIAL1_TXO/PPS: J12.3, J2.2, ZED_CONTROL.2
- removed net N$1: D3.A, R12.1
- removed net N$17: D5.BLU-C, R1.1
- removed net N$2: D1.A, R11.1
- removed net N$26: D8.A, R24.2
- removed net N$27: D10.A, R25.2
- removed net N$29: D11.A, R26.2
- removed net NMEA-RX: BLUETOOTH_BROADCAST.6, SERIAL1_CONNECTION.6
- removed net NMEA-TX: BLUETOOTH_BROADCAST.3, DUAL_OUTPUT.1, SERIAL1_CONNECTION.3
- removed net VIN: C9.1, D2.5, D5.BLU-A, D6.5, D7.C, D9.C, J7.1, MEAS.2, U10.VDD
- removed net ZED-RXI1: J15.2, R9D.2, SERIAL1_CONNECTION.5
- removed net ZED-TXO1: J15.1, R3.2, SERIAL1_CONNECTION.2
- new net CHG_LED_RES: D5.BLU-C, J7.2, R1.1
- new net ESP_13/POWER_CTRL: D1.A, R22.1, R24.2, U5.MOSI_H/IO13
- new net ESP_14/SETUP_BUTTON: J7.3, S2.1, S4.1, U5.SCK_H/IO14
- new net ESP_15/ICM_!CS!: Q9.D, R47.1, U5.CS0_H/IO15
- new net ESP_18/SCK: J16.CLK/SCK, Q3.D, U5.SCK_V/IO18
- new net ESP_19/CIPO: J16.DAT0/SDO, Q10.D, R49.1, U5.MISO_V/IO19
- new net ESP_2/MUX_A: U1.A, U5.IO2
- new net ESP_23/COPI: J16.CMD/SDI, Q4.D, U5.MOSI_V/IO23
- new net ESP_26/DAC2: U1.X3, U5.IO26
- new net ESP_27: U5.IO27
- new net ESP_4/MUX_B: U1.B, U5.IO4
- new net ESP_5: U5.CS0_V/IO5
- new net ESP_I16/ZED-TXO1: J15.1, R2D.2, U1.X0, U5.IO16
- new net ESP_I34/ZED_TX_READY: J6.1, R3D.2, U5.I34
- new net ESP_I36/ICM_INT: Q7.D, R45.1, U5.SENSOR_VP/I36
- new net ESP_I39/ADC39: U1.Y3, U5.SENSOR_VN/I39
- new net ESP_O17/ZED-RXI1: J15.2, R19.2, R2C.2, U1.Y0
- new net EXTERNAL_DATA_IN: J12.2, J2.3, U1.Y
- new net EXTERNAL_DATA_OUT: J12.3, J2.2, U1.X
- new net EXTINT_LV: R9B.1, U3.EXTINT
- new net ICM-20948-LV_!CS!: Q9.S, R46.1, U13.!CS
- new net ICM-20948-LV_#_1.8V: C52.1, C53.1, Q10.G, Q3.G, Q4.G, Q7.G, Q9.G, R40.2, R41.2, R44.2, R46.2, R48.2, U13.VDD, U13.VDDIO, U14.OUT
- new net ICM-20948-LV_INT: Q7.S, R44.1, U13.INT
- new net ICM-20948-LV_SCK: Q3.S, R40.1, U13.SCL/SCLK
- new net ICM-20948-LV_SDI: Q4.S, R41.1, U13.SDA/SDI
- new net ICM-20948-LV_SDO: Q10.S, R48.1, U13.AD0/SDO
- new net N$15: C22.1, C23.2, Q1G1.D, Q1G2.G, R26.1
- new net N$6: R19.1, U5.IO17
- new net N$8: C20.2, Q1G1.G, R24.1
- new net POWER_BTN: C23.1, D1.C, J7.4, R31.1, S1.1, S3.1
- new net VOUT: C20.1, C6.1, Q1G2.D, R22.2, U2.EN, U2.IN
- new net V_RAW: C22.2, C9.1, D3.C, D7.C, J11.4, J9.1, Q1G2.S, R26.2, R31.2, U10.VDD
- new net V_USB: D2.5, D3.A, D5.BLU-A, D6.5, D9.C, MEAS.2
- new net ZED_!RESET!: J6.3, R3B.2
- new net ZED_!RESET!_LV: R3B.1, U3.!RESET!
- new net ZED_EXTINT: R9B.2, U1.Y1
- net 3.3V: now also C3.1, C54.1, R45.2, R47.2, R49.2, U1.VCC, U14.EN, U14.IN; no longer R12.2
- net ESP_21/SDA: now also R2B.2, U1.Y2; no longer R9C.2
- net ESP_22/SCL: now also R2A.2, U1.X2; no longer R9B.2
- net ESP_26/ZED_TX_READY_LV: now also R3D.1; no longer R9A.1
- net FENCE_LV: now also R4D.1; no longer R4A.2
- net GND: now also C3.2, C51.2, C52.2, C53.2, C54.2, J7.1, Q1G1.S, S1.2, S2.2, S3.2, S4.2, U1.GND, U1.INH, U1.VEE, U13.GND, U14.GND; no longer D1.C, D10.C, D11.C, D12.C, D8.C, J6.1
- net N$30: now also C51.1, U13.REGOUT; no longer D12.A, R34.2
- net PPS: now also R9A.1; no longer R2A.1
- net RTK_LV: now also R4C.1; no longer R4B.2
- net RX2_LV: now also R4B.1; no longer R4C.2
- net RXLV: now also R2C.1; no longer R9D.1
- net SCL_LV: now also R2A.1; no longer R9B.1
- net SDA_LV: now also R2B.1; no longer R9C.1
- net TX2_LV: now also R4A.1; no longer R4D.2
- net TXLV: now also R2D.1; no longer R3.1
- net ZED-RXI2: now also R4B.2; no longer BLUETOOTH_BROADCAST.4, R4C.1
- net ZED-TXO2: now also R4A.2; no longer BLUETOOTH_BROADCAST.1, R4D.1
- net ZED_!SAFE!: now also J6.4, R3A.2; no longer J18.3, R2C.2
- net ZED_!SAFE!_LV: now also R3A.1; no longer R2C.1
- net ZED_D_SEL: now also J6.2, R3C.2; no longer J18.5, R2B.2
- net ZED_D_SEL_LV: now also R3C.1; no longer R2B.1
- net ZED_FENCE_STAT: now also R4D.2; no longer R4A.1
- net ZED_PPS_STAT: now also J6.5, R9A.2, U1.X1; no longer J18.4, R11.2, R2A.2, ZED_CONTROL.1
- net ZED_RTK_STAT: now also R4C.2; no longer D3.C, R4B.1
Other:
- note added: "3uA Hibernate"
- note added: "600mA Max 55uA Quiescent"
- note added: "80uA Quiescent"
- note added: "860nA Quiescent"
- note added: "Controller In Peripheral Out (CIPO)"
- note added: "Controller Out Peripheral In (COPI)"
- note added: "External Data Port"
- note added: "ICM-20948 IMU"
- note added: "Level Shifting"
- note added: "Maintains GNSS data/almanac"
- note added: "Power Select"
- note added: "R19 prevents potential serial contention with Data Port"
- note added: "SP6214-1.8V ---------------- Iout (max): 100mA Vin (max): 7.0V Vdrop (max): 250mV Iq: 65uA"
- note added: "System Power"
- note added: "USB For ZED-F9P"
- note added: "Voltage Regulator"
- note added: "u-blox ZED-F9P"
- note removed: "Base Status"
- note removed: "Bluetooth"
- note removed: "Close DUAL_OUTPUT jumper to output NMEA Serial1 to both Bluetooth and external Serial1 port."
- note removed: "Default: Bluetooth will broadcast NMEA. Move switch to 'RTCM' to use Bluetooth as radio connection between RTK units for RTCM corrections."
- note removed: "Default: Data Port Outputs Serial/NMEA Move switch to 'PPS/Reset' to connect Pulse-Per-Second to TX pin and ZED-Reset to RX pin"
- note removed: "Default: ZED-Serial1 NMEA connected to Bluetooth. Move switch to 'Ext Cntr' to connect external 'Data' connector to ZED-Serial1."
- note removed: "Ext Cntr"
- note removed: "NMEA"
- note removed: "PPS/Reset"
- note removed: "RTCM"
- note removed: "RTK Solution: Off: None Blinking: Float On: Fixed"
- note removed: "Serial Config NMEA Out"
- note removed: "Serial NMEA"
- note removed: "USB For ZED-F9P Power Switch"
- note removed: "Ublox ZED-F9P"
- note removed: "≤1000mm"
- note removed: "≤100mm"
- note removed: "≤20mm"
- moved on the sheet: C17, C18, C4, C5, C6, C8, C9, D4, D5, D6, D7, J10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

Commit message: Update soft power switch MOSFET
Parts:
- Q1: value DMC2700UDM -> SIL2308-TP; device SparkFun-DiscreteSemi:MOSFET_COMPLIMENTARY_PAIR-DMC2700UDM -> SparkFun-DiscreteSemi:MOSFET_COMPLIMENTARY_PAIR-SIL2308
Changed lines of the file:
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@@
 <part name="R9" library="SparkFun-Resistors" deviceset="33OHM_RA" device="-1206-1/16W-5%" value="33"/>
 <part name="J6" library="SparkFun-Connectors" deviceset="CONN_05" device="NO_SILK"/>
-<part name="Q1" library="SparkFun-DiscreteSemi" deviceset="MOSFET_COMPLIMENTARY_PAIR" device="-DMC2700UDM" value="DMC2700UDM"/>
+<part name="Q1" library="SparkFun-DiscreteSemi" deviceset="MOSFET_COMPLIMENTARY_PAIR" device="-SIL2308" value="SIL2308-TP"/>
 <part name="C20" library="SparkFun-Capacitors" deviceset="10UF" device="-0603-6.3V-20%" value="10uF"/>
 <part name="R22" library="SparkFun-Resistors" deviceset="100KOHM" device="-0603-1/10W-1%" value="100k"/>
