File: Hardware/Production/SparkFun GPS RTK Surveyor-Panel.brd (EAGLE design)
At the start: 226.8 x 137.8 mm, 585 parts, among them J13 Internal, J16 microSD, J17 Qwiic Right Angle, J19 External, J20 USB Female Type C Connector, J21 Power Switch, J24 Start Base, J25 USB Female Type C Connector, J3 USB Female Type C Connector, J32 microSD, J34 Qwiic Right Angle, J36 Internal, J37 External, J38 USB Female Type C Connector, J39 Power Switch, J4 External, J42 Start Base, J43 USB Female Type C Connector, J5 USB Female Type C Connector, J50 microSD, J52 Qwiic Right Angle, J54 Internal, J6 Start Base, J7 Power Switch, Q1 MBT3904DW1T1, Q2 MBT3904DW1T1, Q3 MBT3904DW1T1, U1 3.3V, U10 MCP73833, U11 CH340C, U12 MAX17048, U13 3.3V, U14 MCP73833, U15 3.3V, U16 U-BLOX_ZED-F9P, U17 ESP-WROOM-32NARROW, U18 CH340C, U19 MAX17048, U2 3.3V, U20 3.3V, U21 MCP73833, U3 U-BLOX_ZED-F9P, U4 3.3V, U5 ESP-WROOM-32NARROW, U6 CH340C, U7 MAX17048, U8 U-BLOX_ZED-F9P, U9 ESP-WROOM-32NARROW

Commit message: Update panel files to v1.6 PCB
Parts:
- added D37: PRTR5V0U2F, SparkFun-IC-Power:SOT886
- added D38: (no value), SparkFun-LED:LED-TRICOLOR-5050
- added D39: PESD0402, SparkFun-DiscreteSemi:0402
- BT1, BT2, BT3: value LIPO-OUTLINE1100 -> LIPO-OUTLINE1000
- D13, D25: value Yellow -> (none); device SparkFun-LED:LED-0603 -> SparkFun-LED:LED-TRICOLOR-5050
- D14, D26: value WHITE -> PESD0402; device SparkFun-LED:LED-0603 -> SparkFun-DiscreteSemi:0402
- D15: value PRTR5V0U2F -> WHITE; device SparkFun-IC-Power:SOT886 -> SparkFun-LED:LED-0603
- D16: value RED -> PRTR5V0U2F; device SparkFun-LED:LED-0603 -> SparkFun-IC-Power:SOT886
- D17: value 3A/10V/280mV -> RED; device SparkFun-DiscreteSemi:SOD-323 -> SparkFun-LED:LED-0603
- D18, D31: value GREEN -> 3A/10V/280mV; device SparkFun-LED:LED-0603 -> SparkFun-DiscreteSemi:SOD-323
- D21, D33: value BLUE -> GREEN
- D22: value 3A/10V/280mV -> BLUE; device SparkFun-DiscreteSemi:SOD-323 -> SparkFun-LED:LED-0603
- D23: value RGB -> 3A/10V/280mV; device SparkFun-LED:PLCC-6-LED -> SparkFun-DiscreteSemi:SOD-323
- D27: value PRTR5V0U2F -> Yellow; device SparkFun-IC-Power:SOT886 -> SparkFun-LED:LED-0603
- D28: value RED -> WHITE
- D29: value 3A/10V/280mV -> PRTR5V0U2F; device SparkFun-DiscreteSemi:SOD-323 -> SparkFun-IC-Power:SOT886
- D30: value GREEN -> RED
- D34: value 3A/10V/280mV -> GREEN; device SparkFun-DiscreteSemi:SOD-323 -> SparkFun-LED:LED-0603
- D35: value RGB -> BLUE; device SparkFun-LED:PLCC-6-LED -> SparkFun-LED:LED-0603
- D36: value PRTR5V0U2F -> 3A/10V/280mV; device SparkFun-IC-Power:SOT886 -> SparkFun-DiscreteSemi:SOD-323
- D5: value RGB -> Yellow; device SparkFun-LED:PLCC-6-LED -> SparkFun-LED:LED-0603
- U1: value 3.3V -> ESP-WROOM-3232D-NARROW; device SparkFun-IC-Power:SOT23-5 -> SparkFun-RF:ESP-WROOM-32D-NARROW
- U11, U18: value CH340C -> MAX17048; device SparkFun-IC-Comms:SO016 -> SparkFun-IC-Power:DFN-8
- U12, U19: value MAX17048 -> 3.3V; device SparkFun-IC-Power:DFN-8 -> SparkFun-IC-Power:SOT23-5
- U13, U20: value 3.3V -> MCP73833; device SparkFun-IC-Power:SOT23-5 -> SparkFun-IC-Power:DFN-10
- U14, U21: value MCP73833 -> ESP-WROOM-3232D-NARROW; device SparkFun-IC-Power:DFN-10 -> SparkFun-RF:ESP-WROOM-32D-NARROW
- U17, U9: value ESP-WROOM-32NARROW -> CH340C; device SparkFun-RF:ESP-WROOM-32-NARROW -> SparkFun-IC-Comms:SO016
- U5: value ESP-WROOM-32NARROW -> 3.3V; device SparkFun-RF:ESP-WROOM-32-NARROW -> SparkFun-IC-Power:SOT23-5
- moved U5 96.4 mm to (111.8, 38.0), flipped to the top
- moved U1 96.3 mm to (34.2, 95.1), flipped to the bottom
- moved D14 93.5 mm to (22.0, 10.7), turned to 180 degrees
- moved D26 93.5 mm to (90.7, 10.7), turned to 180 degrees
- moved D29 85.7 mm to (170.3, 13.9), flipped to the top
- moved D17 63.9 mm to (85.1, 35.4), flipped to the top, turned to 0 degrees
- moved U12 61.3 mm to (102.9, 45.7), flipped to the top, turned to 90 degrees
- moved U19 61.3 mm to (171.6, 45.7), flipped to the top, turned to 90 degrees
- moved D13 59.5 mm to (51.9, 35.2)
- moved D5 59.5 mm to (108.5, 53.9)
- moved D25 59.5 mm to (120.7, 35.2)
- moved U13 58.6 mm to (85.1, 101.5), flipped to the bottom
- moved U20 58.6 mm to (153.8, 101.5), flipped to the bottom
- moved D22 50.8 mm to (108.5, 61.5), turned to 0 degrees
- moved D31 45.5 mm to (160.1, 99.0), flipped to the bottom, turned to 90 degrees
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Connections:
- removed net N$10 (its old number): D5.CG, R6.1
- removed net N$14 (its old number): D5.CR, R8.1
- removed net N$16 (its old number): D16.A, R42.2
- new net N$15: D15.A, R31.1
- new net N$7: D13.3, R6.1
- new net N$8: D13.2, R8.1
- net 3.3V: now also U1.2; no longer U5.2
- net 3.3V1: now also U14.2, U5.5, U9.16, U9.4; no longer U1.5, U11.16, U11.4, U9.2
- net 3.3V2: now also U17.16, U17.4, U21.2; no longer U17.2, U18.16, U18.4
- net 5V1: now also U5.1, U5.3; no longer U1.1, U1.3
- net BACKUP1: now also U12.5; no longer U13.5
- net BACKUP2: now also U19.5; no longer U20.5
- net CHG_LED1: now also U13.3; no longer U14.3
- net CHG_LED2: now also U20.3; no longer U21.3
- net D+2: now also D16.4; no longer D15.4
- net D+3: now also U9.5; no longer U11.5
- net D+4: now also D29.4; no longer D27.4
- net D+5: now also D37.4, U17.5; no longer D36.4, U18.5
- net D-2: now also D16.6; no longer D15.6
- net D-3: now also U9.6; no longer U11.6
- net D-4: now also D29.6; no longer D27.6
- net D-5: now also D37.6, U17.6; no longer D36.6, U18.6
- net ESP32_!DTR1: now also U9.13; no longer U11.13
- net ESP32_!DTR2: now also U17.13; no longer U18.13
- net ESP32_!RTS1: now also U9.14; no longer U11.14
- net ESP32_!RTS2: now also U17.14; no longer U18.14
- net ESP32_EN: now also U1.3; no longer U5.3
- net ESP32_EN1: now also U14.3; no longer U9.3
- net ESP32_EN2: now also U21.3; no longer U17.3
- net ESP32_RXI: now also U1.34; no longer U5.34
- net ESP32_RXI1: now also U14.34, U9.2; no longer U11.2, U9.34
- net ESP32_RXI2: now also U17.2, U21.34; no longer U17.34, U18.2
- net ESP32_TXO: now also U1.35; no longer U5.35
- net ESP32_TXO1: now also U14.35, U9.3; no longer U11.3, U9.35
- net ESP32_TXO2: now also U17.3, U21.35; no longer U17.35, U18.3
- net ESP_0/BOOT: now also U1.25; no longer U5.25
- net ESP_0/BOOT1: now also U14.25; no longer U9.25
- net ESP_0/BOOT2: now also U21.25; no longer U17.25
- net ESP_1: now also U14.13; no longer U9.13
- net ESP_12/LED_BLUETOOTH: now also U1.14; no longer U5.14
- net ESP_12/LED_BLUETOOTH1: now also U14.14; no longer U9.14
- net ESP_12/LED_BLUETOOTH2: now also U21.14; no longer U17.14
- net ESP_13/LED_100CM: now also U1.16; no longer U5.16
- net ESP_13/LED_100CM1: now also U14.16; no longer U9.16
- net ESP_13/LED_100CM2: now also U21.16; no longer U17.16
- net ESP_14: now also U1.13; no longer U5.13
- net ESP_15/LED_10CM: now also U1.23; no longer U5.23
- net ESP_15/LED_10CM1: now also U14.23; no longer U9.23
- net ESP_15/LED_10CM2: now also U21.23; no longer U17.23
- net ESP_16/BT_RXI: now also U1.27; no longer U5.27
- net ESP_16/BT_RXI1: now also U14.27; no longer U9.27
- net ESP_16/BT_RXI2: now also U21.27; no longer U17.27
- net ESP_17/BT_TXO: now also U1.28; no longer U5.28
- net ESP_17/BT_TXO1: now also U14.28; no longer U9.28
- net ESP_17/BT_TXO2: now also U21.28; no longer U17.28
- net ESP_18/SD_SCK: now also U1.30; no longer U5.30
- net ESP_18/SD_SCK1: now also U14.30; no longer U9.30
- net ESP_18/SD_SCK2: now also U21.30; no longer U17.30
- net ESP_19/SD_CIPO: now also U1.31; no longer U5.31
- net ESP_19/SD_CIPO1: now also U14.31; no longer U9.31
- net ESP_19/SD_CIPO2: now also U21.31; no longer U17.31
- net ESP_2: now also U21.13; no longer U17.13
- net ESP_2/LED_1CM: now also U1.24; no longer U5.24
- net ESP_2/LED_1CM1: now also U14.24; no longer U9.24
- net ESP_2/LED_1CM2: now also U21.24; no longer U17.24
- net ESP_21/SDA: now also U1.33; no longer U5.33
- net ESP_21/SDA1: now also U11.8, U14.33; no longer U12.8, U9.33
- net ESP_21/SDA2: now also U18.8, U21.33; no longer U17.33, U19.8
- net ESP_22/SCL: now also U1.36; no longer U5.36
- net ESP_22/SCL1: now also U11.7, U14.36; no longer U12.7, U9.36
- net ESP_22/SCL2: now also U18.7, U21.36; no longer U17.36, U19.7
- net ESP_23/SD_COPI: now also U1.37; no longer U5.37
- net ESP_23/SD_COPI1: now also U14.37; no longer U9.37
- net ESP_23/SD_COPI2: now also U21.37; no longer U17.37
- net ESP_25/SD_!CS!: now also U1.10; no longer U5.10
- net ESP_25/SD_!CS!1: now also U14.10; no longer U9.10
- net ESP_25/SD_!CS!2: now also U21.10; no longer U17.10
- net ESP_26/ZED_TX_READY: now also U1.11; no longer U5.11
- net ESP_26/ZED_TX_READY1: now also U14.11; no longer U9.11
- net ESP_26/ZED_TX_READY2: now also U21.11; no longer U17.11
- net ESP_27/ZED_!RESET!: now also U1.12; no longer U5.12
- net ESP_27/ZED_!RESET!1: now also U14.12; no longer U9.12
- net ESP_27/ZED_!RESET!2: now also U21.12; no longer U17.12
- net ESP_32/PWR_LVL_RED: now also D13.5, U1.8; no longer D5.AR, U5.8
- net ESP_32/PWR_LVL_RED1: now also D25.5, U14.8; no longer D23.AR, U9.8
- net ESP_32/PWR_LVL_RED2: now also D38.5, U21.8; no longer D35.AR, U17.8
- net ESP_33/PWR_LVL_GRN: now also D13.4, U1.9; no longer D5.AG, U5.9
- net ESP_33/PWR_LVL_GRN1: now also D25.4, U14.9; no longer D23.AG, U9.9
- net ESP_33/PWR_LVL_GRN2: now also D38.4, U21.9; no longer D35.AG, U17.9
- net ESP_36/BATT_ALRT: now also U1.4; no longer U5.4
- net ESP_36/BATT_ALRT1: now also U11.5, U14.4; no longer U12.5, U9.4
- net ESP_36/BATT_ALRT2: now also U18.5, U21.4; no longer U17.4, U19.5
- net ESP_4/LED_BASE_STAT: now also U1.26; no longer U5.26
- net ESP_4/LED_BASE_STAT1: now also U14.26; no longer U9.26
- net ESP_4/LED_BASE_STAT2: now also U21.26; no longer U17.26
- net ESP_5/SWITCH_BASE_SELECT: now also U1.29; no longer U5.29
- net ESP_5/SWITCH_BASE_SELECT1: now also U14.29; no longer U9.29
- net ESP_5/SWITCH_BASE_SELECT2: now also U21.29; no longer U17.29
- net ESP_D1+2: now also D37.3; no longer D36.3
- net ESP_D1-2: now also D37.1; no longer D36.1
- net ESP_I1: now also U14.5; no longer U9.5
- net ESP_I2: now also U14.6; no longer U9.6
- net ESP_I3: now also U14.7; no longer U9.7
- net ESP_I34: now also U1.6; no longer U5.6
- net ESP_I35: now also U1.7; no longer U5.7
- net ESP_I39: now also U1.5; no longer U5.5
- net ESP_I4: now also U21.5; no longer U17.5
- net ESP_I5: now also U21.6; no longer U17.6
- net ESP_I6: now also U21.7; no longer U17.7
- net GND: now also D14.2, U1.1, U1.15, U1.38, U1.GND1, U1.GNDT1, U1.GNDT2, U1.GNDT3, U1.GNDT4, U1.GNDT5, U1.GNDT6, U1.GNDT7, U1.GNDT8; no longer U5.1, U5.15, U5.38, U5.GND
- net GND1: now also D16.2, D17.C, D22.C, D26.2, D5.C, U11.4, U11.6, U11.9, U12.2, U13.11, U13.5, U14.1, U14.15, U14.38, U14.GND1, U14.GNDT1, U14.GNDT2, U14.GNDT3, U14.GNDT4, U14.GNDT5, U14.GNDT6, U14.GNDT7, U14.GNDT8, U5.2; no longer D13.C, D15.2, D16.C, D18.C, U1.2, U12.1, U12.4, U12.6, U12.9, U13.2, U14.11, U14.5, U9.15, U9.38, U9.GND
- net GND2: now also D27.C, D29.2, D34.C, D35.C, D37.2, D39.2, U18.4, U18.6, U18.9, U19.2, U20.11, U20.5, U21.1, U21.15, U21.38, U21.GND1, U21.GNDT1, U21.GNDT2, U21.GNDT3, U21.GNDT4, U21.GNDT5, U21.GNDT6, U21.GNDT7, U21.GNDT8; no longer D25.C, D27.2, D28.C, D31.C, D36.2, U17.15, U17.38, U17.GND, U19.1, U19.4, U19.6, U19.9, U20.2, U21.11, U21.5
- net GPS_ANT1: now also D14.1
- net GPS_ANT2: now also D26.1
- net GPS_ANT3: now also D39.1
- net N$17: now also D17.A, R42.2; no longer D5.CB, R1.1
- net N$18: now also D19.A; no longer D18.A
- net N$19: now also D20.A; no longer D19.A
- net N$20: now also D21.A; no longer D20.A
- net N$23: now also D23.A; no longer D22.A
- net N$28: now also D22.A; no longer D21.A
- net N$33: now also R59.1, U13.8; no longer D23.CG, R56.1
- net N$34: now also D25.1, R55.1; no longer D23.CR, R57.1
- net N$35: now also D25.3, R56.1; no longer D23.CB, R55.1
- net N$36: now also D25.2, R57.1; no longer R59.1, U14.8
- net N$37: now also D27.A; no longer D25.A
- net N$40: now also D28.A; no longer D26.A
- net N$42: now also D30.A; no longer D28.A
- net N$43: now also D32.A; no longer D30.A
- net N$44: now also D33.A; no longer D31.A
- net N$45: now also D34.A; no longer D32.A
- net N$48: now also D36.A; no longer D34.A
- net N$49: now also D35.A; no longer D33.A
- net N$51: now also R89.1, U20.8; no longer D35.CG, R86.1
- net N$52: now also D38.1, R85.1; no longer D35.CR, R87.1
- net N$53: now also D38.3, R86.1; no longer D35.CB, R85.1
- net N$54: now also D38.2, R87.1; no longer R89.1, U21.8
- net N$6: now also D13.1, R1.1; no longer D13.A, R19.1
- net N$9: now also D5.A, R19.1; no longer D14.A, R31.1
- net PROG2: now also U13.6; no longer U14.6
- net PROG3: now also U20.6; no longer U21.6
- net UNP_D+1: now also D16.3; no longer D15.3
- net UNP_D+2: now also D29.3; no longer D27.3
- net UNP_D-1: now also D16.1; no longer D15.1
- net UNP_D-2: now also D29.1; no longer D27.1
- net VIN: now also D13.6; no longer D5.AB
- net VIN1: now also D16.5, D18.C, D23.C, D25.6, U13.1, U13.2; no longer D15.5, D17.C, D22.C, D23.AB, U14.1, U14.2
- net VIN2: now also D29.5, D31.C, D36.C, D37.5, D38.6, U20.1, U20.2; no longer D27.5, D29.C, D34.C, D35.AB, D36.5, U21.1, U21.2
- net V_BATT1: now also D18.A, U11.2, U11.3, U12.1, U13.10, U13.9; no longer D17.A, U12.2, U13.1, U13.3, U14.10, U14.9
- net V_BATT2: now also D31.A, U18.2, U18.3, U19.1, U20.10, U20.9; no longer D29.A, U19.2, U20.1, U20.3, U21.10, U21.9
- net ZED_RTK_STAT1: now also D15.C; no longer D14.C
- net ZED_RTK_STAT2: now also D28.C; no longer D26.C
Routing:
- net N$8: track 0.00 -> 4.41 mm
- net N$33: track 1.91 -> 5.65 mm
- net N$51: track 1.91 -> 5.65 mm
- net ZED-TXO6: track 93.2 -> 89.7 mm, vias 3 -> 4
- net ZED-TXO4: track 93.2 -> 89.7 mm, vias 3 -> 4
- net ZED-TXO2: track 93.2 -> 89.7 mm, vias 3 -> 4
- net N$6: track 1.28 -> 4.50 mm
- net CHG_LED2: track 100.1 -> 96.9 mm
- net CHG_LED1: track 100.1 -> 96.9 mm
- net CHG_LED: track 100.1 -> 96.9 mm
- net ZED_RTK_STAT1: track 34.2 -> 37.3 mm
- net ZED_RTK_STAT: track 34.2 -> 37.3 mm
- net ZED_RTK_STAT2: track 34.2 -> 37.3 mm
- net N$7: track 0.00 -> 3.10 mm
- net N$34: track 1.74 -> 4.50 mm
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Other:
- board size 226.8 x 137.8 mm -> 219.3 x 144.2 mm
- board text added: "v16"
- board text removed: "v15"
